File: hardware/HixButton.brd (EAGLE design)
At the start: 16 parts, among them J1 FTDI, J3 XH2P

Commit message: hardware update
Parts:
- added C1: 100nF, rcl:C1206
- added L1: GRN, led:CHIPLED_1206
- added L2: RED, led:CHIPLED_1206
- added R3, R4: 10K, rcl:R1206
- added U1: TPS3839L30, 0_HixField:SOT23
- added WAKE: XH2P, 0_HixField:XH2P
- added X1: MINI-USB_SHIELD5P4-32005-400, con-cypressindustries:32005-400
- C2: value 47μF -> 1uF; device rcl:SMC_A -> rcl:C1206
- moved C2 116.1 mm to (-152.4, -320.0), turned to 0 degrees
- renumbered AWAKE to JMP1, J3 to LIFEPO4
Connections:
- removed net N$7: R10.1, S3.1, U$2.RST
- new net N$10: C2.1, R4.2, X1.1
- new net N$11: L1.A, L2.A, R4.1
- new net N$12: L2.C
- new net N$13: L1.C
- new net N$5: R10.1, S3.2, U$2.RST, WAKE.1
- new net N$6: R3.2
- new net N$9: S3.1, U1.2, WAKE.2
- net 3.3V: now also C1.1, U1.3; no longer C2.+
- net GND: now also C1.2, C2.2, R3.1, U1.1, X1.4; no longer C2.-, S3.2
Routing:
- net N$7: track 1.77 -> 0.40 mm
- net GND: track 1.14 -> 0.56 mm

Commit message: updated hardware board and schematic
Parts:
- removed U$2: ESP8266(ESP12E)V2, 0_HixField:ESP8266(ESP12E)
- removed U$3: LED_RGB, 0_HixField:LED_PL9823-F5
- added U2: CN3058E, 0_HixField:SOP8
- added U3: ESP8266(ESP12E)V2, 0_HixField:ESP8266(ESP12E)
- added U4: LED_RGBWS2812_5050, 0_HixField:LED_5050
- R3: value 10K -> 1.2K
- R4: value 10K -> 330
- moved X1 466.0 mm to (77.5, 67.3), turned to 180 degrees
- moved L1 464.8 mm to (77.5, 74.9), turned to 90 degrees
- moved C2 453.1 mm to (67.3, 76.2), turned to 180 degrees
- moved R4 452.0 mm to (67.3, 58.4), turned to 180 degrees
- moved L2 447.9 mm to (77.5, 59.7), turned to 90 degrees
- moved R3 443.1 mm to (67.3, 72.4), turned to 180 degrees
- moved C1 427.8 mm to (67.3, 62.2), turned to 180 degrees
- moved LIFEPO4 420.4 mm to (61.0, 74.5), turned to 90 degrees
- moved U1 420.1 mm to (52.1, 67.3)
- moved JMP1 397.9 mm to (12.7, 74.9), turned to 180 degrees
- moved WAKE 394.4 mm to (12.7, 66.0)
- moved R1 391.4 mm to (31.8, 67.3), flipped to the bottom
- moved C3 343.4 mm to (52.1, 71.1), turned to 0 degrees
- moved S3 337.3 mm to (59.7, 67.3), turned to 270 degrees
- moved J1 325.9 mm to (19.1, 63.5), turned to 0 degrees
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Connections:
- removed net N$10: C2.1, R4.2, X1.1
- new net VIN: C2.1, R4.2, U2.4, X1.1
- net 3.3V: now also U2.5, U2.8, U3.VCC, U4.3; no longer U$2.VCC, U$3.VCC
- net GND: now also U2.1, U2.3, U3.GND, U4.1; no longer U$2.GND, U$3.GND
- net N$1: now also U3.GPIO15_CS_TXD2; no longer U$2.GPIO15_CS_TXD2
- net N$12: now also U2.7
- net N$13: now also U2.6
- net N$2: now also U3.GPIO2_TXD1; no longer U$2.GPIO2_TXD1
- net N$3: now also U3.GPIO0_FLASH; no longer U$2.GPIO0_FLASH
- net N$4: now also U3.GPIO4_SDA; no longer U$2.GPIO4_SDA
- net N$5: now also U3.RST; no longer U$2.RST
- net N$6: now also U2.2
- net N$8: now also U3.ENABLE; no longer U$2.ENABLE
- net RGB: now also U3.GPIO5_SCL, U4.2; no longer U$2.GPIO5_SCL, U$3.DIN
- net RXD: now also U3.GPIO1_TXD0; no longer U$2.GPIO1_TXD0
- net TXD: now also U3.GPIO3_RXD0; no longer U$2.GPIO3_RXD0
Routing:
- net 3.3V: track 1.23 -> 0.00 mm
- net RGB: track 1.20 -> 0.00 mm, vias 2 -> 0
- net GND: track 0.56 -> 0.00 mm
- net N$7: track 0.40 -> 0.00 mm, vias 3 -> 0
- net N$8: track 0.17 -> 0.00 mm, vias 1 -> 0
Other:
- board outline added: 75.4 x 22.3 mm
- board text removed: "HixButton v1.0.0"
- board text removed: "HixField (C) 2020"

Commit message: updated hardware
Parts:
- removed S4: PROG, 0_HixField:SMDPUSHBTN_TYPE1
- added C10: 1uF, rcl:C1206
- added C4: 100nF, rcl:C1206
- added C7, C8, C9: 100μF, rcl:SMC_A
- added PROG: (no value), jumper:SJ
- C2: value 1uF -> 100nF
- C5: value 100nF -> 100μF; device rcl:C1206 -> rcl:SMC_A
- C6: value 680μF/6.3V -> 100μF; device 0_HixField:ELKO_RADIAL_STRAIGHT_4P_8D_9H -> rcl:SMC_A
- U1: value TPS3839L30 -> ESP8266(ESP12E)V2; device 0_HixField:SOT23 -> 0_HixField:ESP8266(ESP12E)
- U2: value CN3058E -> TPS3839L30; device 0_HixField:SOP8 -> 0_HixField:SOT23
- U3: value ESP8266(ESP12E)V2 -> CN3058E; device 0_HixField:ESP8266(ESP12E) -> 0_HixField:SOP8
- moved C1 67.6 mm to (6.35, 33.0), turned to 0 degrees
- moved C2 67.1 mm to (6.35, 48.3), turned to 0 degrees
- moved C6 59.5 mm to (6.35, 21.6), turned to 0 degrees
- moved C3 53.6 mm to (6.35, 43.2)
- moved C5 52.4 mm to (6.35, 26.7), flipped to the top, turned to 0 degrees
- moved U3 31.8 mm to (67.3, 67.3), turned to 270 degrees
- moved U1 16.5 mm to (35.6, 67.3), turned to 90 degrees
- moved U2 15.2 mm to (52.1, 67.3), turned to 0 degrees
- renumbered JMP1 to STAYAWAKE
Connections:
- net 3.3V: now also C2.1, C4.1, C5.+, C7.+, C8.+, C9.+, U1.VCC, U2.3, U3.5, U3.8; no longer C5.1, U1.3, U2.5, U2.8, U3.VCC
- net GND: now also C10.2, C4.2, C5.-, C7.-, C8.-, C9.-, PROG.1, U1.GND, U3.1, U3.3; no longer C5.2, S4.2, U1.1, U2.3, U3.GND
- net N$1: now also U1.GPIO15_CS_TXD2; no longer U3.GPIO15_CS_TXD2
- net N$12: now also U3.7; no longer U2.7
- net N$13: now also U3.6; no longer U2.6
- net N$2: now also U1.GPIO2_TXD1; no longer U3.GPIO2_TXD1
- net N$3: now also PROG.2, U1.GPIO0_FLASH; no longer S4.1, U3.GPIO0_FLASH
- net N$4: now also U1.GPIO4_SDA; no longer U3.GPIO4_SDA
- net N$5: now also U1.RST; no longer U3.RST
- net N$6: now also U3.2; no longer U2.2
- net N$8: now also U1.ENABLE; no longer U3.ENABLE
- net N$9: now also U2.2; no longer U1.2
- net RGB: now also U1.GPIO5_SCL; no longer U3.GPIO5_SCL
- net RXD: now also U1.GPIO1_TXD0; no longer U3.GPIO1_TXD0
- net TXD: now also U1.GPIO3_RXD0; no longer U3.GPIO3_RXD0
- net VIN: now also C10.1, U3.4; no longer C2.1, U2.4

Commit message: updated sch and board layout
Parts:
- removed X1: MINI-USB_SHIELD5P4-32005-400, con-cypressindustries:32005-400
- R3: value 1.2K -> 5.6K
- U4: value LED_RGBWS2812_5050 -> WS2812
- moved C9 73.4 mm to (50.8, 64.8)
- moved C8 71.4 mm to (50.8, 67.3)
- moved C7 69.4 mm to (50.8, 69.8)
- moved C3 67.9 mm to (71.8, 61.6), turned to 90 degrees
- moved C6 67.5 mm to (50.8, 72.4)
- moved C5 65.6 mm to (50.8, 74.9)
- moved J1 62.2 mm to (81.3, 63.5)
- moved C4 61.9 mm to (61.0, 67.3), turned to 90 degrees
- moved WAKE 52.3 mm to (64.8, 61.0), turned to 270 degrees
- moved PROG 47.6 mm to (57.1, 59.7)
- moved C2 45.7 mm to (50.8, 59.1)
- moved STAYAWAKE 44.5 mm to (57.1, 74.9)
- moved C1 42.7 mm to (31.8, 67.3), flipped to the bottom
- moved R4 15.3 mm to (71.8, 73.0), turned to 90 degrees
- moved L2 12.1 mm to (76.2, 71.8)
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Connections:
- removed net VIN: C10.1, R4.2, U3.4, X1.1
- new net 5.0V: C10.1, J1.5V, R4.2, U3.4
- net 3.3V: no longer J1.5V
- net GND: no longer X1.4
Other:
- board size 75.4 x 22.3 mm -> 54.6 x 20.1 mm

Commit message: update board
Parts:
- moved C4 1.91 mm to (62.9, 67.3)
- moved C9 1.91 mm to (50.8, 66.7)
- moved C8 1.27 mm to (50.8, 68.6)
- moved U4 1.27 mm to (67.3, 67.3), turned to 270 degrees
- moved C5 0.64 mm to (50.8, 74.3)
- moved C7 0.64 mm to (50.8, 70.5)
- moved U2 0.64 mm to (50.8, 62.9), turned to 90 degrees
- moved C2 0.63 mm to (50.8, 59.7)
- turned R3 to 90 degrees
- turned S3 to 90 degrees
