File: hardware/HixButton.brd (EAGLE design)
At the start: 55.9 x 20.1 mm, 28 parts, among them J1 FTDIFTDI_ANGLED, U1 ESP8266(ESP12E)V2, U2 TPS3839L30, U3 CN3058E, U4 WS2812

Commit message: added sj 3d model
Parts:
- PROG, STAYAWAKE: device jumper:SJ -> 0_HixField:SJ
Changed lines of the file:
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@@
 <attribute name="NAME" x="81.407" y="58.547" size="0.762" layer="25" rot="R180" align="center"/>
 </element>
-<element name="STAYAWAKE" library="jumper" library_urn="urn:adsk.eagle:library:252" package="SJ" package3d_urn="urn:adsk.eagle:package:15471/1" value="" x="57.15" y="74.93" smashed="yes">
+<element name="STAYAWAKE" library="0_HixField" library_urn="urn:adsk.eagle:library:13392178" package="SJ" package3d_urn="urn:adsk.eagle:package:25478059/2" value="" x="57.15" y="74.93" smashed="yes">
 <attribute name="NAME" x="52.832" y="76.2" size="0.762" layer="25" ratio="10"/>
 <attribute name="POPULARITY" value="33" x="81.28" y="5.08" size="1.778" layer="27" display="off"/>
@@
 <attribute name="NAME" x="60.96" y="60.071" size="0.762" layer="25" rot="R270" align="center"/>
 </element>
-<element name="PROG" library="jumper" library_urn="urn:adsk.eagle:library:252" package="SJ" package3d_urn="urn:adsk.eagle:package:15471/1" value="" x="57.15" y="60.198" smashed="yes">
+<element name="PROG" library="0_HixField" library_urn="urn:adsk.eagle:library:13392178" package="SJ" package3d_urn="urn:adsk.eagle:package:25478059/2" value="" x="57.15" y="60.198" smashed="yes">
 <attribute name="NAME" x="55.753" y="58.039" size="0.762" layer="25" ratio="10"/>
 <attribute name="POPULARITY" value="33" x="57.15" y="60.198" size="1.778" layer="27" display="off"/>
+<attribute name="SPICEPREFIX" value="B" x="57.15" y="60.198" size="1.778" layer="27" display="off"/>
 <attribute name="VALUE" x="57.5501" y="60.198" size="0.02" layer="27"/>
 </element>
